File: Hardware/Hardware.kicad_pcb (KiCad board)
At the start: 4 copper layers, 0 parts

Commit message: added stepfiles
Parts:
- added C1: TBD, Capacitor_SMD:C_0603_1608Metric, F.Cu at (165.2, 99.8)
- added C10: 10u, Capacitor_SMD:C_0603_1608Metric, F.Cu at (107.2, 97.8)
- added C2: TBD, Capacitor_SMD:C_0402_1005Metric, F.Cu at (113.0, 100.0)
- added C3: TBD, Capacitor_SMD:C_0402_1005Metric, F.Cu at (116.4, 103.8)
- added C4: 470p, Capacitor_SMD:C_0402_1005Metric, F.Cu at (118.4, 102.0)
- added C5: 1u, Capacitor_SMD:C_0603_1608Metric, F.Cu at (118.6, 104.8)
- added C6: 100n, Capacitor_SMD:C_0402_1005Metric, F.Cu at (115.2, 97.6)
- added C7: 10u, Capacitor_SMD:C_0603_1608Metric, F.Cu at (112.4, 97.4)
- added C8: 100n, Capacitor_SMD:C_0402_1005Metric, F.Cu at (114.0, 97.6)
- added C9: 100n, Capacitor_SMD:C_0402_1005Metric, F.Cu at (108.8, 98.5)
- added J1: Micro_SD_Card, Connector_Card:microSD_HC_Molex_47219-2001, F.Cu at (270.8, 24.5)
- added J2: USB_C_Receptacle_USB2.0, Connector_USB:USB_C_Receptacle_XKB_U262-16XN-4BVC11, F.Cu at (280.4, 52.0)
- added J3: RJ45_RB1-125B8G1A, Connector_RJ:RJ45_UDE_RB1-125B8G1A, F.Cu at (168.7, 98.5)
- added L1: BLM18PG121SN1D, Inductor_SMD:L_0603_1608Metric, F.Cu at (109.8, 96.6)
- added R1: 47k, Resistor_SMD:R_0603_1608Metric, F.Cu at (281.0, 18.6)
- added R10: 50R, Resistor_SMD:R_0603_1608Metric, F.Cu at (161.8, 85.4)
- added R11: 50R, Resistor_SMD:R_0603_1608Metric, F.Cu at (159.2, 85.4)
- added R12: 50R, Resistor_SMD:R_0603_1608Metric, F.Cu at (156.7, 85.4)
- added R13: 12k1, Resistor_SMD:R_0603_1608Metric, F.Cu at (117.4, 94.8)
- added R14: 10k, Resistor_SMD:R_0603_1608Metric, F.Cu at (180.2, 82.6)
- added R15: 10k, Resistor_SMD:R_0603_1608Metric, F.Cu at (180.4, 103.0)
- added R16: 330R, Resistor_SMD:R_0603_1608Metric, F.Cu at (182.8, 102.2)
- added R17: 330R, Resistor_SMD:R_0603_1608Metric, F.Cu at (182.8, 83.4)
- added R18: 100k, Resistor_SMD:R_0603_1608Metric, F.Cu at (129.6, 106.4)
- added R19: 33R, Resistor_SMD:R_0603_1608Metric, F.Cu at (259.1, 60.4)
- added R2: 47k, Resistor_SMD:R_0603_1608Metric, F.Cu at (281.0, 21.2)
- added R20: 33R, Resistor_SMD:R_0603_1608Metric, F.Cu at (259.1, 62.9)
- added R21: 4k7, Resistor_SMD:R_0603_1608Metric, F.Cu at (123.2, 106.4)
- added R22: 4k7, Resistor_SMD:R_0603_1608Metric, F.Cu at (121.6, 106.4)
- added R23: 1k5, Resistor_SMD:R_0603_1608Metric, F.Cu at (126.4, 106.4)
- added R24: 4k7, Resistor_SMD:R_0603_1608Metric, F.Cu at (128.0, 106.4)
- added R25: 33R, Resistor_SMD:R_0603_1608Metric, F.Cu at (259.0, 56.8)
- added R26: 1k5, Resistor_SMD:R_0603_1608Metric, F.Cu at (124.8, 106.4)
- added R3: 47k, Resistor_SMD:R_0603_1608Metric, F.Cu at (281.0, 23.7)
- added R4: 47k, Resistor_SMD:R_0603_1608Metric, F.Cu at (281.0, 26.2)
- added R5: 47k, Resistor_SMD:R_0603_1608Metric, F.Cu at (281.0, 28.7)
- added R6: 47k, Resistor_SMD:R_0603_1608Metric, F.Cu at (281.1, 31.7)
- added R7: 5k1, Resistor_SMD:R_0603_1608Metric, F.Cu at (280.4, 42.4)
- added R8: 5k1, Resistor_SMD:R_0603_1608Metric, F.Cu at (280.4, 45.6)
- added R9: 50R, Resistor_SMD:R_0603_1608Metric, F.Cu at (164.3, 85.4)
- added U1: STM32F407VET6, Package_QFP:LQFP-100_14x14mm_P0.5mm, F.Cu at (247.9, 60.9)
- added U2: USBLC6-2SC6, Package_TO_SOT_SMD:SOT-23-6, F.Cu at (272.8, 51.8)
- added U3: LAN8742A, Package_DFN_QFN:VQFN-24-1EP_4x4mm_P0.5mm_EP2.5x2.5mm_ThermalVias, F.Cu at (120.5, 98.3)
- added Y1: 25MHz, Crystal:Crystal_SMD_3225-4Pin_3.2x2.5mm, F.Cu at (115.6, 101.0)
Routing:
- net GND: track 0.00 -> 33.1 mm, vias 0 -> 10
- net +3V3: track 0.00 -> 17.0 mm, vias 0 -> 3
- net ETH_RST: track 0.00 -> 12.4 mm
- net ETH_REF_CLK: track 0.00 -> 10.9 mm
- net Net-(U3-VDD1A): track 0.00 -> 8.89 mm
- net /IO/ETH_LED1: track 0.00 -> 7.68 mm, vias 0 -> 1
- net ETH_MDIO: track 0.00 -> 7.25 mm
- net ETH_CRS_DV: track 0.00 -> 6.82 mm
- net ETH_RXD0: track 0.00 -> 6.78 mm
- net Net-(U3-XTAL2): track 0.00 -> 6.46 mm
- net ETH_RXD1: track 0.00 -> 6.32 mm
- net Net-(U3-XTAL1/CLKIN): track 0.00 -> 6.32 mm
- net Net-(J3-PadL2): track 0.00 -> 5.85 mm
- net Net-(U3-VDDCR): track 0.00 -> 5.47 mm
- net /IO/ETH_LED2: track 0.00 -> 5.42 mm, vias 0 -> 1
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- added copper zone on B.Cu, net +3V3
- added copper zone on In1.Cu, net GND
- added copper zone on In2.Cu, net GND
